Commit message: Put ros2 control in Xacro file

File: rb1_ros2_description/xacro/rb1_ros2_base.urdf.xacro (robot description, xacro)
@@ -85,4 +85,27 @@
 	</xacro:sensor_orbbec_astra>
 	<!-- Gazebo ros2 control plugins -->
+    <ros2_control name="diff_drive" type="system">
+      <hardware>
+          <plugin>gazebo_ros2_control/GazeboSystem</plugin>
+      </hardware>
+      <joint name="left_wheel_joint">
+        <command_interface name="velocity">
+          <param name="min">-1</param>
+          <param name="max">1</param>
+        </command_interface>
+        <state_interface name="position"/>
+        <state_interface name="velocity"/>
+        <state_interface name="effort"/>
+      </joint>
+      <joint name="right_wheel_joint">
+        <command_interface name="velocity">
+          <param name="min">-1</param>
+          <param name="max">1</param>
+        </command_interface>
+        <state_interface name="position"/>
+        <state_interface name="velocity"/>
+        <state_interface name="effort"/>
+      </joint>
+    </ros2_control>
 	<!-- <xacro:ros2_control/> -->
 </robot>

Commit message: Modify the joint name to fit current Robot model and joint name in the config file

File: rb1_ros2_description/xacro/rb1_ros2_base.urdf.xacro (robot description, xacro)
@@ -89,5 +89,5 @@
           <plugin>gazebo_ros2_control/GazeboSystem</plugin>
       </hardware>
-      <joint name="left_wheel_joint">
+      <joint name="robot_left_wheel_joint">
         <command_interface name="velocity">
           <param name="min">-1</param>
@@ -98,5 +98,5 @@
         <state_interface name="effort"/>
       </joint>
-      <joint name="right_wheel_joint">
+      <joint name="robot_right_wheel_joint">
         <command_interface name="velocity">
           <param name="min">-1</param>

Commit message: Add ros2 control joint_trajectory in xacro

File: rb1_ros2_description/xacro/rb1_ros2_base.urdf.xacro (robot description, xacro)
@@ -108,4 +108,19 @@
       </joint>
     </ros2_control>
+      <!-- Position Config -->
+    <ros2_control name="elevator" type="system">
+        <hardware>
+            <plugin>gazebo_ros2_control/GazeboSystem</plugin>
+        </hardware>
+        <joint name="robot_elevator_platform_joint">
+            <command_interface name="position">
+            <param name="min">0.00</param>
+            <param name="max">0.05</param>
+            </command_interface>
+            <state_interface name="position"/>
+            <state_interface name="velocity"/>
+            <state_interface name="effort"/>
+        </joint>
+    </ros2_control>
 	<!-- <xacro:ros2_control/> -->
     <gazebo>
