Commit message: Add friction for joint to avoid elevator slide down

File: rb1_ros2_description/urdf/elevator/elevator.urdf.xacro (robot description, xacro)
@@ -60,5 +60,6 @@
 			<child link="${prefix}_platform_link" />
 			<axis xyz="0 0 1"/>
-			<limit effort="10.0" lower="0.0" upper="0.034" velocity="0.5"/>
+			<limit effort="20.0" lower="0.0" upper="0.034" velocity="2.0"/>
+            <dynamics damping="0.1" friction="1.0"/>
 	</joint>
 	<link name="${prefix}_platform_link">
